File: AutoSteerAiO.brd (EAGLE design)
At the start: 114.3 x 99.1 mm, 81 parts, among them IC2 MMA8452Q, J4 CONNECTOR 1x5 PINS, K4 CB1A-P-12V

Commit message: Add files via upload
Routing:
- net N$25: track 66.1 -> 80.1 mm
- net A+5V: track 31.3 -> 36.2 mm
- net GND: vias 77 -> 76
Changed lines of the file:
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@@
 <drawing>
 <settings>
-<setting alwaysvectorfont="no"/>
+<setting alwaysvectorfont="yes"/>
 <setting keepoldvectorfont="yes"/>
 <setting verticaltext="up"/>
 </settings>
-<grid distance="50" unitdist="mil" unit="mil" style="lines" multiple="1" display="yes" altdistance="12.5" altunitdist="mil" altunit="mil"/>
+<grid distance="50" unitdist="mil" unit="mil" style="lines" multiple="1" display="yes" altdistance="25" altunitdist="mil" altunit="mil"/>
 <layers>
 <layer number="1" name="Top" color="4" fill="1" visible="yes" active="yes"/>
@@
 <wire x1="46.355" y1="72.39" x2="31.115" y2="72.39" width="0.1524" layer="21"/>
 <wire x1="31.115" y1="72.39" x2="31.115" y2="89.535" width="0.1524" layer="21"/>
-<text x="39.37" y="74.295" size="1.27" layer="21" font="vector" ratio="14" align="center">ENC28J60</text>
+<text x="39.37" y="75.565" size="1.27" layer="21" font="vector" ratio="14" align="center">ENC28J60</text>
 <text x="38.735" y="91.44" size="1.016" layer="21" font="vector" ratio="14" rot="SR180" align="center">HR911105A</text>
 <text x="9.525" y="78.74" size="0.8128" layer="25" font="vector" ratio="14" rot="R90" align="center">+5V</text>
@@
 <text x="15.875" y="34.925" size="0.7112" layer="25" font="vector" ratio="13" rot="R90" align="center">BLK</text>
 <text x="15.875" y="37.465" size="0.7112" layer="25" font="vector" ratio="13" rot="R90" align="center">BRN</text>
+<wire x1="11.43" y1="65.405" x2="10.795" y2="65.405" width="0.0762" layer="21"/>
+<wire x1="11.43" y1="62.865" x2="10.795" y2="62.865" width="0.0762" layer="21"/>
+<wire x1="10.795" y1="65.405" x2="10.795" y2="64.77" width="0.0762" layer="21"/>
+<wire x1="10.795" y1="62.865" x2="10.795" y2="63.5" width="0.0762" layer="21"/>
+<wire x1="10.795" y1="63.5" x2="10.16" y2="64.135" width="0.0762" layer="21"/>
+<wire x1="11.43" y1="50.165" x2="10.795" y2="50.165" width="0.0762" layer="21"/>
+<wire x1="11.43" y1="47.625" x2="10.795" y2="47.625" width="0.0762" layer="21"/>
+<wire x1="10.795" y1="50.165" x2="10.795" y2="49.53" width="0.0762" layer="21"/>
+<wire x1="10.795" y1="47.625" x2="10.795" y2="48.26" width="0.0762" layer="21"/>
+<wire x1="10.795" y1="48.26" x2="10.16" y2="48.895" width="0.0762" layer="21"/>
+<wire x1="11.43" y1="34.925" x2="10.795" y2="34.925" width="0.0762" layer="21"/>
+<wire x1="11.43" y1="32.385" x2="10.795" y2="32.385" width="0.0762" layer="21"/>
+<wire x1="10.795" y1="34.925" x2="10.795" y2="34.29" width="0.0762" layer="21"/>
+<wire x1="10.795" y1="32.385" x2="10.795" y2="33.02" width="0.0762" layer="21"/>
+<wire x1="10.795" y1="33.02" x2="10.16" y2="33.655" width="0.0762" layer="21"/>
 </plain>
 <attributes>
@@
 <attribute name="CYTRON-PC" value="CN-2600PS-05" x="117.475" y="68.58" size="1.778" layer="27" rot="R90" display="off"/>
 <attribute name="DESC" value="2600 PCB Connector" x="117.475" y="68.58" size="1.778" layer="27" rot="R90" display="off"/>
+<attribute name="LABEL" value="" x="120.396" y="67.183" size="0.762" layer="21" font="vector" ratio="15" rot="R90" align="top-left"/>
 <attribute name="LABEL" value="" x="120.396" y="67.183" size="0.762" layer="51" font="vector" ratio="15" rot="R90" align="top-left"/>
-<attribute name="LABEL" value="" x="120.396" y="67.183" size="0.762" layer="21" font="vector" ratio="15" rot="R90" align="top-left"/>
 <attribute name="LABEL" value="" x="117.475" y="68.58" size="1.778" layer="27" rot="R90" display="off"/>
 <attribute name="MF" value="" x="117.475" y="68.58" size="1.778" layer="27" rot="R90" display="off"/>
@@
 <via x="34.925" y="44.45" extent="1-16" drill="0.508"/>
 <via x="73.66" y="25.4" extent="1-16" drill="0.508"/>
-<via x="38.735" y="76.835" extent="1-16" drill="0.508"/>
+<via x="38.735" y="73.025" extent="1-16" drill="0.508"/>
 <contactref element="J4" pad="1"/>
 <contactref element="JP1" pad="1"/>
@@
 <via x="35.56" y="111.125" extent="1-16" drill="0.508"/>
 <via x="30.48" y="111.125" extent="1-16" drill="0.508"/>
-<via x="38.735" y="87.63" extent="1-16" drill="0.508"/>
-<via x="38.735" y="99.695" extent="1-16" drill="0.508"/>
+<via x="38.735" y="85.725" extent="1-16" drill="0.508"/>
 <wire x1="74.93" y1="62.23" x2="74.93" y2="60.96" width="2.032" layer="16"/>
 <wire x1="17.78" y1="106.68" x2="17.78" y2="88.9" width="0.8128" layer="16"/>
@@
 <contactref element="L1" pad="2"/>
 <contactref element="ADS1115" pad="1"/>
-<wire x1="85.09" y1="66.04" x2="83.82" y2="64.77" width="0.508" layer="1"/>
-<wire x1="83.82" y1="64.77" x2="83.82" y2="61.595" width="0.508" layer="1"/>
-<wire x1="83.82" y1="61.595" x2="77.47" y2="55.245" width="0.508" layer="1"/>
-<wire x1="74.93" y1="55.245" x2="77.47" y2="55.245" width="0.508" layer="1"/>
 <contactref element="C8" pad="2"/>
 <wire x1="87.63" y1="66.04" x2="85.09" y2="66.04" width="0.508" layer="1"/>
 <contactref element="D4" pad="A"/>
-<wire x1="92.71" y1="59.055" x2="92.71" y2="55.88" width="0.508" layer="1"/>
-<wire x1="92.71" y1="59.055" x2="88.9" y2="62.865" width="0.508" layer="1"/>
-<wire x1="87.63" y1="66.04" x2="88.9" y2="64.77" width="0.508" layer="1"/>
-<wire x1="88.9" y1="64.77" x2="88.9" y2="62.865" width="0.508" layer="1"/>
+<wire x1="92.71" y1="58.42" x2="92.71" y2="55.88" width="0.508" layer="1"/>
+<wire x1="92.71" y1="58.42" x2="87.63" y2="63.5" width="0.508" layer="1"/>
+<wire x1="87.63" y1="63.5" x2="87.63" y2="66.04" width="0.508" layer="1"/>
+<wire x1="74.93" y1="55.245" x2="81.915" y2="55.245" width="0.508" layer="1"/>
+<wire x1="81.915" y1="55.245" x2="85.09" y2="52.07" width="0.508" layer="1"/>
+<wire x1="85.09" y1="52.07" x2="90.17" y2="52.07" width="0.508" layer="1"/>
+<wire x1="92.71" y1="54.61" x2="92.71" y2="55.88" width="0.508" layer="1"/>
+<wire x1="92.71" y1="54.61" x2="90.17" y2="52.07" width="0.508" layer="1"/>
 </signal>
 <signal name="N$25">
@@
 <contactref element="PS1" pad="3"/>
 <wire x1="77.47" y1="66.04" x2="74.93" y2="66.04" width="0.508" layer="1"/>
-<wire x1="26.9825" y1="95.25" x2="55.5975" y2="66.635" width="0.6096" layer="16"/>
-<wire x1="23.4265" y1="95.25" x2="26.9825" y2="95.25" width="0.6096" layer="16"/>
 <contactref element="C9" pad="+"/>
 <wire x1="74.93" y1="66.04" x2="74.335" y2="66.635" width="0.6096" layer="1"/>
 <wire x1="74.335" y1="66.635" x2="66.675" y2="66.635" width="0.6096" layer="1"/>
-<wire x1="55.5975" y1="66.635" x2="66.675" y2="66.635" width="0.6096" layer="16"/>
+<wire x1="52.745" y1="66.635" x2="66.675" y2="66.635" width="0.6096" layer="16"/>
+<wire x1="23.4265" y1="95.25" x2="52.0415" y2="66.635" width="0.6096" layer="16"/>
+<wire x1="52.0415" y1="66.635" x2="66.675" y2="66.635" width="0.6096" layer="16"/>
 </signal>
 <signal name="N$3">

Commit message: Add files via upload
Parts:
- moved 0 18.1 mm to (46.4, 25.4), turned to 90 degrees
- moved C12 15.4 mm to (50.8, 33.7), turned to 270 degrees
- moved D2 8.89 mm to (43.2, 90.8)
- moved D3 8.89 mm to (34.3, 90.8)
- moved IC2 7.24 mm to (61.0, 31.1), turned to 90 degrees
- moved C11 5.08 mm to (41.9, 65.4)
- moved PCB1 5.08 mm to (47.6, 32.4)
- moved R16 2.22 mm to (56.5, 81.6)
- moved R17 2.22 mm to (67.3, 81.6)
- moved LED1 1.91 mm to (56.5, 86.4)
- moved LED2 1.91 mm to (67.3, 86.4)
- moved U$5 1.27 mm to (38.7, 102.2)
- moved U$8 1.27 mm to (40.0, 108.0)
- moved C4 0.64 mm to (67.3, 95.2)
- moved PS1 0.25 mm to (24.4, 97.8)
Routing:
- net GND: track 500.4 -> 479.1 mm, vias 76 -> 79
- net A2: track 5.72 -> 24.4 mm
- net +15V: track 149.5 -> 131.5 mm
- net N$25: track 80.1 -> 66.4 mm
- net A1: track 5.72 -> 19.3 mm
- net +5V: track 245.9 -> 233.5 mm
- net +3V3: track 24.8 -> 12.6 mm
- net D6: track 14.8 -> 9.49 mm
- net RST: track 23.7 -> 18.6 mm
- net D8: track 14.8 -> 19.1 mm
- net D2: track 38.8 -> 34.7 mm
- net N$1: track 18.8 -> 15.0 mm
- net D7: track 3.17 -> 6.40 mm
- net SCL: track 102.2 -> 99.9 mm
- net SDA: track 100.5 -> 99.2 mm
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Other:
- board text added: "MMA8542"
- board text removed: "HR911105A"

Commit message: Add files via upload
Parts:
- moved R6 0.63 mm to (59.7, 49.5)
- moved R7 0.63 mm to (62.2, 49.5)
Routing:
- net SCL: track 99.9 -> 99.0 mm
- net N$9: track 15.0 -> 15.7 mm
- net N$1: track 15.0 -> 15.7 mm
Changed lines of the file:
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@@
 <drawing>
 <settings>
-<setting alwaysvectorfont="yes"/>
+<setting alwaysvectorfont="no"/>
 <setting keepoldvectorfont="yes"/>
 <setting verticaltext="up"/>
@@
 <text x="54.61" y="33.02" size="0.7112" layer="25" font="vector" ratio="10" align="center">3V</text>
 <text x="67.31" y="33.02" size="0.7112" layer="25" font="vector" ratio="10" align="center">GND</text>
-<text x="59.69" y="48.895" size="1.016" layer="25" font="vector" ratio="12" rot="R270" align="center">330</text>
-<text x="62.23" y="48.895" size="1.016" layer="25" font="vector" ratio="12" rot="R270" align="center">330</text>
+<text x="59.69" y="49.53" size="1.016" layer="25" font="vector" ratio="12" rot="R270" align="center">330</text>
+<text x="62.23" y="49.53" size="1.016" layer="25" font="vector" ratio="12" rot="R270" align="center">330</text>
 <text x="60.325" y="109.22" size="1.6764" layer="25" font="vector" ratio="14" rot="R180" align="center">GND</text>
 <wire x1="55.245" y1="107.95" x2="60.325" y2="107.95" width="0.508" layer="21"/>
@@
 <text x="67.6275" y="50.165" size="1.016" layer="25" font="vector" ratio="12" rot="R180" align="center">MMA8542</text>
 <text x="14.605" y="80.645" size="0.8128" layer="25" font="vector" ratio="12" rot="R90" align="center">output</text>
-<wire x1="53.975" y1="32.385" x2="55.88" y2="32.385" width="0.1524" layer="21"/>
+<wire x1="53.6575" y1="32.385" x2="55.88" y2="32.385" width="0.1524" layer="21"/>
 <wire x1="55.88" y1="32.385" x2="58.42" y2="32.385" width="0.1524" layer="21"/>
 <wire x1="58.42" y1="32.385" x2="60.96" y2="32.385" width="0.1524" layer="21"/>
@@
 <wire x1="53.34" y1="30.1625" x2="53.34" y2="32.0675" width="0.1524" layer="21"/>
 <wire x1="53.34" y1="32.0675" x2="53.6575" y2="32.385" width="0.1524" layer="21"/>
-<wire x1="53.6575" y1="32.385" x2="53.975" y2="32.385" width="0.1524" layer="21"/>
 <wire x1="55.88" y1="32.385" x2="55.88" y2="29.845" width="0.1524" layer="21"/>
 <wire x1="58.42" y1="32.385" x2="58.42" y2="29.845" width="0.1524" layer="21"/>
@@
 <attribute name="VALUE" x="101.6" y="49.53" size="1.016" layer="25" font="vector" ratio="12" align="center"/>
 </element>
-<element name="R6" library="resistor" library_urn="urn:adsk.eagle:library:348" package="0207/7" package3d_urn="urn:adsk.eagle:package:23493/2" value="330" x="59.69" y="48.895" smashed="yes" rot="R90">
-<attribute name="MF" value="" x="59.69" y="48.895" size="1.778" layer="27" rot="R90" display="off"/>
-<attribute name="MPN" value="" x="59.69" y="48.895" size="1.778" layer="27" rot="R90" display="off"/>
-<attribute name="OC_NEWARK" value="unknown" x="59.69" y="48.895" size="1.778" layer="27" rot="R90" display="off"/>
-</element>
-<element name="R7" library="resistor" library_urn="urn:adsk.eagle:library:348" package="0207/7" package3d_urn="urn:adsk.eagle:package:23493/2" value="330" x="62.23" y="48.895" smashed="yes" rot="R90">
-<attribute name="MF" value="" x="62.23" y="48.895" size="1.778" layer="27" rot="R90" display="off"/>
-<attribute name="MPN" value="" x="62.23" y="48.895" size="1.778" layer="27" rot="R90" display="off"/>
-<attribute name="OC_NEWARK" value="unknown" x="62.23" y="48.895" size="1.778" layer="27" rot="R90" display="off"/>
+<element name="R6" library="resistor" library_urn="urn:adsk.eagle:library:348" package="0207/7" package3d_urn="urn:adsk.eagle:package:23493/2" value="330" x="59.69" y="49.53" smashed="yes" rot="R90">
+<attribute name="MF" value="" x="59.69" y="49.53" size="1.778" layer="27" rot="R90" display="off"/>
+<attribute name="MPN" value="" x="59.69" y="49.53" size="1.778" layer="27" rot="R90" display="off"/>
+<attribute name="OC_NEWARK" value="unknown" x="59.69" y="49.53" size="1.778" layer="27" rot="R90" display="off"/>
+</element>
+<element name="R7" library="resistor" library_urn="urn:adsk.eagle:library:348" package="0207/7" package3d_urn="urn:adsk.eagle:package:23493/2" value="330" x="62.23" y="49.53" smashed="yes" rot="R90">
+<attribute name="MF" value="" x="62.23" y="49.53" size="1.778" layer="27" rot="R90" display="off"/>
+<attribute name="MPN" value="" x="62.23" y="49.53" size="1.778" layer="27" rot="R90" display="off"/>
+<attribute name="OC_NEWARK" value="unknown" x="62.23" y="49.53" size="1.778" layer="27" rot="R90" display="off"/>
 </element>
 <element name="R9" library="resistor" library_urn="urn:adsk.eagle:library:348" package="0207/7" package3d_urn="urn:adsk.eagle:package:23493/2" value="330" x="104.14" y="75.565" smashed="yes" rot="R180">
@@
 <attribute name="CYTRON-PC" value="CN-2600PS-05" x="117.475" y="68.58" size="1.778" layer="27" rot="R90" display="off"/>
 <attribute name="DESC" value="2600 PCB Connector" x="117.475" y="68.58" size="1.778" layer="27" rot="R90" display="off"/>
+<attribute name="LABEL" value="" x="120.396" y="67.183" size="0.762" layer="51" font="vector" ratio="15" rot="R90" align="top-left"/>
 <attribute name="LABEL" value="" x="120.396" y="67.183" size="0.762" layer="21" font="vector" ratio="15" rot="R90" align="top-left"/>
-<attribute name="LABEL" value="" x="120.396" y="67.183" size="0.762" layer="51" font="vector" ratio="15" rot="R90" align="top-left"/>
 <attribute name="LABEL" value="" x="117.475" y="68.58" size="1.778" layer="27" rot="R90" display="off"/>
 <attribute name="MF" value="" x="117.475" y="68.58" size="1.778" layer="27" rot="R90" display="off"/>
@@
 <contactref element="TO_SECTION" pad="1"/>
 <wire x1="74.93" y1="50.165" x2="90.4875" y2="50.165" width="0.4064" layer="1"/>
-<wire x1="62.23" y1="52.705" x2="59.69" y2="55.245" width="0.4064" layer="16"/>
-<wire x1="46.355" y1="55.245" x2="59.69" y2="55.245" width="0.4064" layer="16"/>
+<wire x1="62.23" y1="53.34" x2="60.325" y2="55.245" width="0.4064" layer="16"/>
+<wire x1="46.355" y1="55.245" x2="60.325" y2="55.245" width="0.4064" layer="16"/>
 <wire x1="103.1875" y1="62.865" x2="117.475" y2="62.865" width="0.4064" layer="1"/>
 <wire x1="103.1875" y1="62.865" x2="90.4875" y2="50.165" width="0.4064" layer="1"/>
 <contactref element="MMA8542" pad="SCL"/>
-<wire x1="62.23" y1="57.15" x2="62.23" y2="52.705" width="0.4064" layer="1"/>
+<wire x1="62.23" y1="57.15" x2="62.23" y2="53.34" width="0.4064" layer="1"/>
 </signal>
 <signal name="SDA">
@@
 <contactref element="R6" pad="2"/>
 <contactref element="TO_SECTION" pad="2"/>
-<wire x1="59.69" y1="52.705" x2="56.1975" y2="49.2125" width="0.4064" layer="16"/>
-<wire x1="56.1975" y1="49.2125" x2="51.1175" y2="49.2125" width="0.4064" layer="16"/>
+<wire x1="59.69" y1="53.34" x2="55.5625" y2="49.2125" width="0.4064" layer="16"/>
+<wire x1="55.5625" y1="49.2125" x2="51.1175" y2="49.2125" width="0.4064" layer="16"/>
 <wire x1="51.1175" y1="49.2125" x2="47.625" y2="52.705" width="0.4064" layer="16"/>
 <wire x1="46.355" y1="52.705" x2="47.625" y2="52.705" width="0.4064" layer="16"/>
@@
 <wire x1="90.4875" y1="47.625" x2="74.93" y2="47.625" width="0.4064" layer="1"/>
 <contactref element="MMA8542" pad="SDA"/>
-<wire x1="59.69" y1="57.15" x2="59.69" y2="52.705" width="0.4064" layer="1"/>
+<wire x1="59.69" y1="57.15" x2="59.69" y2="53.34" width="0.4064" layer="1"/>
 <wire x1="51.1175" y1="49.2125" x2="47.625" y2="52.705" width="0.4064" layer="1"/>
 <wire x1="47.625" y1="52.705" x2="46.355" y2="52.705" width="0.4064" layer="1"/>
@@
 <contactref element="IC2" pad="2"/>
 <contactref element="R6" pad="1"/>
-<wire x1="59.69" y1="45.085" x2="59.69" y2="37.465" width="0.4064" layer="1"/>
+<wire x1="59.69" y1="45.72" x2="59.69" y2="37.465" width="0.4064" layer="1"/>
 <wire x1="59.69" y1="37.465" x2="57.15" y2="34.925" width="0.4064" layer="1"/>
 <wire x1="57.15" y1="34.925" x2="57.15" y2="31.115" width="0.4064" layer="1"/>
@@
 <contactref element="IC2" pad="3"/>
 <contactref element="R7" pad="1"/>
-<wire x1="62.23" y1="36.195" x2="62.23" y2="45.085" width="0.4064" layer="1"/>
+<wire x1="62.23" y1="36.195" x2="62.23" y2="45.72" width="0.4064" layer="1"/>
 <wire x1="59.69" y1="31.115" x2="59.69" y2="33.655" width="0.4064" layer="1"/>
 <wire x1="59.69" y1="33.655" x2="62.23" y2="36.195" width="0.4064" layer="1"/>

Commit message: Add files via upload
Parts:
- moved INT 7.36 mm to (27.6, 80.3)
- moved D1 5.08 mm to (110.5, 88.9)
- moved ON/OFF 1.27 mm to (117.5, 105.4), turned to 180 degrees
- moved RESET 0.63 mm to (27.3, 73.7)
Routing:
- net GND: track 479.1 -> 461.3 mm, vias 79 -> 84
- net V+: track 6.29 -> 11.4 mm
- net D2: track 34.7 -> 29.9 mm
- net N$26: track 79.4 -> 77.2 mm
- net N$5: track 41.9 -> 40.3 mm
- net RST: track 18.6 -> 18.0 mm

Commit message: Add files via upload
Parts:
- moved +5V 0.32 mm to (12.7, 79.1)
- moved GND34 0.32 mm to (12.7, 82.2)
Other:
- board text removed: "BAT+"
- board text removed: "BAT-"

Commit message: Add files via upload
Routing:
- net GND: vias 84 -> 85
Changed lines of the file:
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@@
 <attribute name="CYTRON-PC" value="CN-2600PS-05" x="117.475" y="68.58" size="1.778" layer="27" rot="R90" display="off"/>
 <attribute name="DESC" value="2600 PCB Connector" x="117.475" y="68.58" size="1.778" layer="27" rot="R90" display="off"/>
+<attribute name="LABEL" value="" x="120.396" y="67.183" size="0.762" layer="21" font="vector" ratio="15" rot="R90" align="top-left"/>
 <attribute name="LABEL" value="" x="120.396" y="67.183" size="0.762" layer="51" font="vector" ratio="15" rot="R90" align="top-left"/>
-<attribute name="LABEL" value="" x="120.396" y="67.183" size="0.762" layer="21" font="vector" ratio="15" rot="R90" align="top-left"/>
 <attribute name="LABEL" value="" x="117.475" y="68.58" size="1.778" layer="27" rot="R90" display="off"/>
 <attribute name="MF" value="" x="117.475" y="68.58" size="1.778" layer="27" rot="R90" display="off"/>
@@
 <wire x1="11.3665" y1="30.099" x2="10.16" y2="31.3055" width="0.6096" layer="1"/>
 <wire x1="14.9225" y1="75.565" x2="10.16" y2="70.8025" width="0.6096" layer="1"/>
-<wire x1="13.7313125" y1="88.9" x2="12.7" y2="88.9" width="0.4064" layer="1"/>
-<wire x1="17.3381125" y1="92.5068" x2="13.7313125" y2="88.9" width="0.4064" layer="1"/>
+<wire x1="15.0013125" y1="88.9" x2="12.7" y2="88.9" width="0.4064" layer="1"/>
+<wire x1="18.6081125" y1="92.5068" x2="15.0013125" y2="88.9" width="0.4064" layer="1"/>
 <wire x1="51.435" y1="80.01" x2="38.9382" y2="92.5068" width="0.4064" layer="1"/>
-<wire x1="38.9382" y1="92.5068" x2="17.3381125" y2="92.5068" width="0.4064" layer="1"/>
+<wire x1="38.9382" y1="92.5068" x2="18.6081125" y2="92.5068" width="0.4064" layer="1"/>
 <wire x1="61.9125" y1="80.01" x2="63.5" y2="81.5975" width="0.4064" layer="1"/>
 <wire x1="51.435" y1="80.01" x2="61.9125" y2="80.01" width="0.4064" layer="1"/>
@@
 <contactref element="C10" pad="1"/>
 <via x="60.325" y="111.125" extent="1-16" drill="0.508"/>
-<via x="35.56" y="111.125" extent="1-16" drill="0.508"/>
 <wire x1="17.78" y1="106.68" x2="17.78" y2="88.9" width="0.8128" layer="16"/>
 <contactref element="MMA8542" pad="GND"/>
@@
 <via x="10.16" y="110.49" extent="1-16" drill="0.508"/>
 <via x="119.38" y="110.49" extent="1-16" drill="0.508"/>
+<via x="38.1" y="116.84" extent="1-16" drill="0.508"/>
+<via x="33.02" y="116.84" extent="1-16" drill="0.508"/>
 </signal>
 <signal name="D5">
