File: AutoSteerAiO.sch (EAGLE design)
At the start: 82 parts, among them IC2 MMA8452Q, J4 CONNECTOR 1x5 PINS, K4 CB1A-P-12V

Commit message: Add files via upload
Connections:
- net HIGH.: no longer R4.1
- net LOW.: now also R4.1
Changed lines of the file:
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@@
 <segment>
 <pinref part="WAS_D" gate="G$1" pin="3"/>
-<wire x1="177.8" y1="241.3" x2="190.5" y2="241.3" width="0.1524" layer="91"/>
 <label x="177.8" y="241.3" size="1.778" layer="95"/>
 <pinref part="R11" gate="G$1" pin="1"/>
-<pinref part="R4" gate="G$1" pin="1"/>
-<wire x1="190.5" y1="241.3" x2="203.2" y2="241.3" width="0.1524" layer="91"/>
-<wire x1="190.5" y1="248.92" x2="190.5" y2="241.3" width="0.1524" layer="91"/>
-<junction x="190.5" y="241.3"/>
+<wire x1="177.8" y1="241.3" x2="203.2" y2="241.3" width="0.1524" layer="91"/>
 </segment>
 </net>
@@
 <pinref part="R10" gate="G$1" pin="1"/>
 <wire x1="177.8" y1="243.84" x2="187.96" y2="243.84" width="0.1524" layer="91"/>
-<wire x1="203.2" y1="254" x2="187.96" y2="254" width="0.1524" layer="91"/>
+<wire x1="203.2" y1="254" x2="190.5" y2="254" width="0.1524" layer="91"/>
+<wire x1="190.5" y1="254" x2="187.96" y2="254" width="0.1524" layer="91"/>
 <wire x1="187.96" y1="254" x2="187.96" y2="243.84" width="0.1524" layer="91"/>
+<pinref part="R4" gate="G$1" pin="1"/>
+<wire x1="190.5" y1="248.92" x2="190.5" y2="254" width="0.1524" layer="91"/>
+<junction x="190.5" y="254"/>
 </segment>
 </net>

Commit message: Add files via upload
silkscreen
Parts:
- +5V, +5V1, GND33, GND34: MPN HEF4093BT,653 -> (none); OC_NEWARK 70R5288 -> unknown
- U$3: MPN (none) -> ATSAMD10C13A-SSNT; OC_NEWARK (none) -> 90Y6375
Changed lines of the file:
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@@
 <part name="+5V" library="wirepad" library_urn="urn:adsk.eagle:library:412" deviceset="2,15/1,0" device="" package3d_urn="urn:adsk.eagle:package:30831/1">
 <attribute name="MF" value=""/>
-<attribute name="MPN" value="HEF4093BT,653"/>
-<attribute name="OC_NEWARK" value="70R5288"/>
+<attribute name="MPN" value=""/>
+<attribute name="OC_NEWARK" value="unknown"/>
 </part>
 <part name="+5V1" library="wirepad" library_urn="urn:adsk.eagle:library:412" deviceset="2,15/1,0" device="" package3d_urn="urn:adsk.eagle:package:30831/1">
 <attribute name="MF" value=""/>
-<attribute name="MPN" value="HEF4093BT,653"/>
-<attribute name="OC_NEWARK" value="70R5288"/>
+<attribute name="MPN" value=""/>
+<attribute name="OC_NEWARK" value="unknown"/>
 </part>
 <part name="GND33" library="wirepad" library_urn="urn:adsk.eagle:library:412" deviceset="2,15/1,0" device="" package3d_urn="urn:adsk.eagle:package:30831/1">
 <attribute name="MF" value=""/>
-<attribute name="MPN" value="HEF4093BT,653"/>
-<attribute name="OC_NEWARK" value="70R5288"/>
+<attribute name="MPN" value=""/>
+<attribute name="OC_NEWARK" value="unknown"/>
 </part>
 <part name="GND34" library="wirepad" library_urn="urn:adsk.eagle:library:412" deviceset="2,15/1,0" device="" package3d_urn="urn:adsk.eagle:package:30831/1">
 <attribute name="MF" value=""/>
-<attribute name="MPN" value="HEF4093BT,653"/>
-<attribute name="OC_NEWARK" value="70R5288"/>
+<attribute name="MPN" value=""/>
+<attribute name="OC_NEWARK" value="unknown"/>
 </part>
 <part name="GND25" library="supply1" library_urn="urn:adsk.eagle:library:371" deviceset="GND" device=""/>
@@
 <attribute name="OC_NEWARK" value="unknown"/>
 </part>
-<part name="U$3" library="#Motor Drivers" deviceset="MD10C" device=""/>
+<part name="U$3" library="#Motor Drivers" deviceset="MD10C" device="">
+<attribute name="MF" value=""/>
+<attribute name="MPN" value="ATSAMD10C13A-SSNT"/>
+<attribute name="OC_NEWARK" value="90Y6375"/>
+</part>
 </parts>
 <sheets>
@@
 <attribute name="MPN" x="147.32" y="231.14" size="1.778" layer="96" display="off"/>
 </instance>
-<instance part="U$3" gate="G$1" x="144.78" y="139.7" smashed="yes"/>
+<instance part="U$3" gate="G$1" x="144.78" y="139.7" smashed="yes">
+<attribute name="OC_NEWARK" x="144.78" y="139.7" size="1.778" layer="96" display="off"/>
+<attribute name="MF" x="144.78" y="139.7" size="1.778" layer="96" display="off"/>
+<attribute name="MPN" x="144.78" y="139.7" size="1.778" layer="96" display="off"/>
+</instance>
 </instances>
 <busses>

Commit message: Add files via upload
Parts:
- removed PS2: VX7805-1000, #VX7805-500:VX7805-500
- added U1: VX7805-1000, #VX7805-1000:VX7805-1000
Connections:
- net +5V: now also U1.+VOUT/GND; no longer PS2.+VOUT
- net GND: now also U1.GND/-VOUT; no longer PS2.GND
- net N$26: now also U1.+VIN; no longer PS2.+VIN
Other:
- moved on the sheet: C10, C16, LED2, R17

Commit message: Add files via upload
wrong footprint VX7805-1000 it can fit but will come out with PCB
Parts:
- U1: OC_NEWARK (none) -> unknown
Changed lines of the file:
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@@
 <attribute name="OC_NEWARK" value="90Y6375"/>
 </part>
-<part name="U1" library="#VX7805-1000" deviceset="VX7805-1000" device=""/>
+<part name="U1" library="#VX7805-1000" deviceset="VX7805-1000" device="">
+<attribute name="MF" value=""/>
+<attribute name="MPN" value=""/>
+<attribute name="OC_NEWARK" value="unknown"/>
+</part>
 </parts>
 <sheets>
@@
 <attribute name="NAME" x="99.0437" y="244.612709375" size="1.78026875" layer="95"/>
 <attribute name="VALUE" x="99.023" y="226.0304" size="1.78318125" layer="96"/>
+<attribute name="OC_NEWARK" x="111.76" y="236.22" size="1.778" layer="96" display="off"/>
+<attribute name="MPN" x="111.76" y="236.22" size="1.778" layer="96" display="off"/>
 </instance>
 </instances>

Commit message: Add files via upload
Removed capacitor after the VX7805 regulator, same as in datasheet https://www.cui.com/product/resource/vx78-500.pdf
Figure 4
Parts:
- removed C16, C9: 1000uF, SparkFun-Capacitors:1000UF-RADIAL-5MM-25V-20%
Connections:
- net +5V: no longer C16.+
- net GND: no longer C16.-, C9.-
- net N$25: no longer C9.+
Other:
- moved on the sheet: C7, C8, L1
Changed lines of the file:
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@@
 <?xml version="1.0" encoding="utf-8"?>
 <!DOCTYPE eagle SYSTEM "eagle.dtd">
-<eagle version="9.3.1">
+<eagle version="9.3.2">
 <drawing>
 <settings>
@@
 <attribute name="OC_NEWARK" value="unknown"/>
 </part>
-<part name="C9" library="SparkFun-Capacitors" library_urn="urn:adsk.eagle:library:510" deviceset="1000UF" device="-RADIAL-5MM-25V-20%" package3d_urn="urn:adsk.eagle:package:37412/1" value="1000uF">
-<attribute name="MF" value=""/>
-<attribute name="MPN" value=""/>
-<attribute name="OC_NEWARK" value="unknown"/>
-</part>
-<part name="C16" library="SparkFun-Capacitors" library_urn="urn:adsk.eagle:library:510" deviceset="1000UF" device="-RADIAL-5MM-25V-20%" package3d_urn="urn:adsk.eagle:package:37412/1" value="1000uF">
-<attribute name="MF" value=""/>
-<attribute name="MPN" value=""/>
-<attribute name="OC_NEWARK" value="unknown"/>
-</part>
 <part name="U$3" library="#Motor Drivers" deviceset="MD10C" device="">
 <attribute name="MF" value=""/>
@@
 <attribute name="VALUE" x="231.14" y="203.2" size="1.778" layer="96"/>
 </instance>
-<instance part="L1" gate="G$1" x="271.78" y="223.52" smashed="yes" rot="R90">
-<attribute name="NAME" x="275.59" y="222.0214" size="1.778" layer="95" rot="R180"/>
-<attribute name="VALUE" x="275.59" y="226.822" size="1.778" layer="96" rot="R180"/>
-<attribute name="OC_NEWARK" x="271.78" y="223.52" size="1.778" layer="96" display="off"/>
-<attribute name="MF" x="271.78" y="223.52" size="1.778" layer="96" display="off"/>
-<attribute name="MPN" x="271.78" y="223.52" size="1.778" layer="96" display="off"/>
+<instance part="L1" gate="G$1" x="261.62" y="223.52" smashed="yes" rot="R90">
+<attribute name="NAME" x="265.43" y="222.0214" size="1.778" layer="95" rot="R180"/>
+<attribute name="VALUE" x="265.43" y="226.822" size="1.778" layer="96" rot="R180"/>
+<attribute name="OC_NEWARK" x="261.62" y="223.52" size="1.778" layer="96" display="off"/>
+<attribute name="MF" x="261.62" y="223.52" size="1.778" layer="96" display="off"/>
+<attribute name="MPN" x="261.62" y="223.52" size="1.778" layer="96" display="off"/>
 </instance>
 <instance part="AGND1" gate="1" x="226.06" y="266.954" smashed="yes">
@@
 <attribute name="MPN" x="218.44" y="223.52" size="1.778" layer="96" display="off"/>
 </instance>
-<instance part="C7" gate="G$1" x="264.16" y="215.9" smashed="yes" rot="R180">
-<attribute name="NAME" x="262.255" y="214.63" size="1.778" layer="95" rot="R180"/>
-<attribute name="VALUE" x="267.97" y="220.0275" size="1.778" layer="96" rot="R180"/>
-<attribute name="OC_NEWARK" x="264.16" y="215.9" size="1.778" layer="96" display="off"/>
-<attribute name="MF" x="264.16" y="215.9" size="1.778" layer="96" display="off"/>
-<attribute name="MPN" x="264.16" y="215.9" size="1.778" layer="96" display="off"/>
-</instance>
-<instance part="C8" gate="G$1" x="279.4" y="215.9" smashed="yes" rot="R180">
-<attribute name="NAME" x="277.495" y="214.63" size="1.778" layer="95" rot="R180"/>
-<attribute name="VALUE" x="283.21" y="220.0275" size="1.778" layer="96" rot="R180"/>
-<attribute name="OC_NEWARK" x="279.4" y="215.9" size="1.778" layer="96" display="off"/>
-<attribute name="MF" x="279.4" y="215.9" size="1.778" layer="96" display="off"/>
-<attribute name="MPN" x="279.4" y="215.9" size="1.778" layer="96" display="off"/>
+<instance part="C7" gate="G$1" x="254" y="215.9" smashed="yes" rot="R180">
+<attribute name="NAME" x="257.175" y="214.63" size="1.778" layer="95" rot="R180"/>
+<attribute name="VALUE" x="257.81" y="220.0275" size="1.778" layer="96" rot="R180"/>
+<attribute name="OC_NEWARK" x="254" y="215.9" size="1.778" layer="96" display="off"/>
+<attribute name="MF" x="254" y="215.9" size="1.778" layer="96" display="off"/>
+<attribute name="MPN" x="254" y="215.9" size="1.778" layer="96" display="off"/>
+</instance>
+<instance part="C8" gate="G$1" x="269.24" y="215.9" smashed="yes" rot="R180">
+<attribute name="NAME" x="267.335" y="214.63" size="1.778" layer="95" rot="R180"/>
+<attribute name="VALUE" x="273.05" y="220.0275" size="1.778" layer="96" rot="R180"/>
+<attribute name="OC_NEWARK" x="269.24" y="215.9" size="1.778" layer="96" display="off"/>
+<attribute name="MF" x="269.24" y="215.9" size="1.778" layer="96" display="off"/>
+<attribute name="MPN" x="269.24" y="215.9" size="1.778" layer="96" display="off"/>
 </instance>
 <instance part="C6" gate="G$1" x="213.36" y="215.9" smashed="yes" rot="R180">
@@
 <attribute name="MPN" x="144.78" y="167.64" size="1.778" layer="96" display="off"/>
 </instance>
-<instance part="C9" gate="G$1" x="254" y="218.44" smashed="yes">
-<attribute name="NAME" x="255.143" y="218.9226" size="1.778" layer="95"/>
-<attribute name="VALUE" x="255.143" y="213.8426" size="1.778" layer="96"/>
-<attribute name="OC_NEWARK" x="254" y="218.44" size="1.778" layer="96" display="off"/>
-<attribute name="MF" x="254" y="218.44" size="1.778" layer="96" display="off"/>
-<attribute name="MPN" x="254" y="218.44" size="1.778" layer="96" display="off"/>
-</instance>
-<instance part="C16" gate="G$1" x="149.86" y="231.14" smashed="yes">
-<attribute name="NAME" x="145.923" y="234.1626" size="1.778" layer="95"/>
-<attribute name="VALUE" x="151.003" y="226.5426" size="1.778" layer="96"/>
-<attribute name="OC_NEWARK" x="149.86" y="231.14" size="1.778" layer="96" display="off"/>
-<attribute name="MF" x="149.86" y="231.14" size="1.778" layer="96" display="off"/>
-<attribute name="MPN" x="149.86" y="231.14" size="1.778" layer="96" display="off"/>
-</instance>
 <instance part="U$3" gate="G$1" x="144.78" y="139.7" smashed="yes">
 <attribute name="OC_NEWARK" x="144.78" y="139.7" size="1.778" layer="96" display="off"/>
@@
 <wire x1="139.7" y1="236.22" x2="139.7" y2="238.76" width="0.1524" layer="91"/>
 <junction x="139.7" y="238.76"/>
-<wire x1="139.7" y1="238.76" x2="149.86" y2="238.76" width="0.1524" layer="91"/>
-<wire x1="149.86" y1="238.76" x2="154.94" y2="238.76" width="0.1524" layer="91"/>
+<wire x1="139.7" y1="238.76" x2="154.94" y2="238.76" width="0.1524" layer="91"/>
 <wire x1="154.94" y1="238.76" x2="154.94" y2="215.9" width="0.1524" layer="91"/>
 <pinref part="C10" gate="G$1" pin="2"/>
 <wire x1="134.62" y1="236.22" x2="134.62" y2="238.76" width="0.1524" layer="91"/>
 <junction x="134.62" y="238.76"/>
-<pinref part="C16" gate="G$1" pin="+"/>
-<wire x1="149.86" y1="233.68" x2="149.86" y2="238.76" width="0.1524" layer="91"/>
-<junction x="149.86" y="238.76"/>
 <pinref part="U1" gate="G$1" pin="+VOUT/GND"/>
 </segment>
@@
 <junction x="134.62" y="218.44"/>
 <pinref part="C10" gate="G$1" pin="1"/>
-<pinref part="C16" gate="G$1" pin="-"/>
-<wire x1="149.86" y1="226.06" x2="149.86" y2="218.44" width="0.1524" layer="91"/>
-<wire x1="149.86" y1="218.44" x2="139.7" y2="218.44" width="0.1524" layer="91"/>
-<junction x="139.7" y="218.44"/>
 </segment>
 <segment>
@@
 <pinref part="C8" gate="G$1" pin="1"/>
 <wire x1="233.68" y1="210.82" x2="254" y2="210.82" width="0.1524" layer="91"/>
-<wire x1="254" y1="210.82" x2="264.16" y2="210.82" width="0.1524" layer="91"/>
-<wire x1="264.16" y1="210.82" x2="279.4" y2="210.82" width="0.1524" layer="91"/>
-<wire x1="279.4" y1="210.82" x2="279.4" y2="213.36" width="0.1524" layer="91"/>
+<wire x1="254" y1="210.82" x2="269.24" y2="210.82" width="0.1524" layer="91"/>
+<wire x1="269.24" y1="210.82" x2="269.24" y2="213.36" width="0.1524" layer="91"/>
 <pinref part="C7" gate="G$1" pin="1"/>
-<wire x1="264.16" y1="213.36" x2="264.16" y2="210.82" width="0.1524" layer="91"/>
-<junction x="264.16" y="210.82"/>
+<wire x1="254" y1="213.36" x2="254" y2="210.82" width="0.1524" layer="91"/>
+<junction x="254" y="210.82"/>
 <pinref part="GND31" gate="1" pin="GND"/>
 <wire x1="233.68" y1="208.28" x2="233.68" y2="210.82" width="0.1524" layer="91"/>
 <junction x="233.68" y="210.82"/>
-<pinref part="C9" gate="G$1" pin="-"/>
-<wire x1="254" y1="213.36" x2="254" y2="210.82" width="0.1524" layer="91"/>
-<junction x="254" y="210.82"/>
 </segment>
 <segment>
@@
 <net name="A+5V" class="0">
 <segment>
-<wire x1="279.4" y1="223.52" x2="279.4" y2="220.98" width="0.1524" layer="91"/>
-<wire x1="279.4" y1="223.52" x2="279.4" y2="226.06" width="0.1524" layer="91"/>
-<junction x="279.4" y="223.52"/>
-<label x="279.4" y="226.06" size="1.778" layer="95"/>
+<wire x1="269.24" y1="223.52" x2="269.24" y2="220.98" width="0.1524" layer="91"/>
+<wire x1="269.24" y1="223.52" x2="269.24" y2="226.06" width="0.1524" layer="91"/>
+<junction x="269.24" y="223.52"/>
+<label x="269.24" y="226.06" size="1.778" layer="95"/>
 <pinref part="L1" gate="G$1" pin="2"/>
-<wire x1="276.86" y1="223.52" x2="279.4" y2="223.52" width="0.1524" layer="91"/>
+<wire x1="266.7" y1="223.52" x2="269.24" y2="223.52" width="0.1524" layer="91"/>
 <pinref part="C8" gate="G$1" pin="2"/>
 </segment>
@@
 <segment>
 <pinref part="L1" gate="G$1" pin="1"/>
-<wire x1="266.7" y1="223.52" x2="264.16" y2="223.52" width="0.1524" layer="91"/>
+<wire x1="256.54" y1="223.52" x2="254" y2="223.52" width="0.1524" layer="91"/>
 <pinref part="C7" gate="G$1" pin="2"/>
-<wire x1="264.16" y1="223.52" x2="254" y2="223.52" width="0.1524" layer="91"/>
+<wire x1="254" y1="223.52" x2="248.92" y2="223.52" width="0.1524" layer="91"/>
 <pinref part="PS1" gate="G$1" pin="+VOUT"/>
-<wire x1="254" y1="223.52" x2="248.92" y2="223.52" width="0.1524" layer="91"/>
-<wire x1="264.16" y1="220.98" x2="264.16" y2="223.52" width="0.1524" layer="91"/>
-<junction x="264.16" y="223.52"/>
-<pinref part="C9" gate="G$1" pin="+"/>
 <wire x1="254" y1="220.98" x2="254" y2="223.52" width="0.1524" layer="91"/>
 <junction x="254" y="223.52"/>

Commit message: Add files via upload
changed the diodes
Parts:
- D2, D3: value 1N4004 -> 1N5400; device diode:1N4004 -> diode:1N5400
Changed lines of the file:
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@@
 <part name="GND3" library="supply1" library_urn="urn:adsk.eagle:library:371" deviceset="GND" device=""/>
 <part name="P+2" library="supply1" library_urn="urn:adsk.eagle:library:371" deviceset="+15V" device=""/>
-<part name="D2" library="diode" library_urn="urn:adsk.eagle:library:210" deviceset="1N4004" device="" package3d_urn="urn:adsk.eagle:package:43336/1">
+<part name="D2" library="diode" library_urn="urn:adsk.eagle:library:210" deviceset="1N5400" device="" package3d_urn="urn:adsk.eagle:package:43365/2">
 <attribute name="MF" value=""/>
 <attribute name="MPN" value=""/>
 <attribute name="OC_NEWARK" value="unknown"/>
 </part>
-<part name="D3" library="diode" library_urn="urn:adsk.eagle:library:210" deviceset="1N4004" device="" package3d_urn="urn:adsk.eagle:package:43336/1">
+<part name="D3" library="diode" library_urn="urn:adsk.eagle:library:210" deviceset="1N5400" device="" package3d_urn="urn:adsk.eagle:package:43365/2">
 <attribute name="MF" value=""/>
 <attribute name="MPN" value=""/>

Commit message: Add files via upload
changed footprint for inductor
Parts:
- added C9: .1uF, resistor:C-EU050-024X044
- L1: device rcl:L-EU0204/7 -> rcl:L-EU0207/10
Connections:
- net +5V: now also C9.2
- net GND: now also C9.1
Other:
- moved on the sheet: C6, C7, C8, L1
