File: AutoSteerAiO.sch (EAGLE design)
At the start: 81 parts, among them IC2 MMA8452Q, J4 CONNECTOR 1x5 PINS, K4 CB1A-P-12V, U1 VX7805-1000

Commit message: Add files via upload
Other:
- moved on the sheet: +5V, +5V1, 0, 15V1, 15V2, ADS1115, AUTO-SWITCH, AUX_A/D, C1, C10, C11, C12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

Commit message: Add files via upload
Parts:
- removed R15: 47, resistor:R-EU_0207/7
Connections:
- removed net PO: AUTO-SWITCH.3, IMP-SWITCH.3, R15.1, STEER-SWITCH.3
- net +15V: now also AUTO-SWITCH.3, IMP-SWITCH.3, STEER-SWITCH.3; no longer R15.2
Changed lines of the file:
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@@
 <layer number="91" name="Nets" color="2" fill="1" visible="yes" active="yes"/>
 <layer number="92" name="Busses" color="1" fill="1" visible="yes" active="yes"/>
-<layer number="93" name="Pins" color="2" fill="1" visible="yes" active="yes"/>
+<layer number="93" name="Pins" color="2" fill="1" visible="no" active="yes"/>
 <layer number="94" name="Symbols" color="4" fill="1" visible="yes" active="yes"/>
 <layer number="95" name="Names" color="7" fill="1" visible="yes" active="yes"/>
@@
 <attribute name="OC_NEWARK" value="unknown"/>
 </part>
-<part name="R15" library="resistor" library_urn="urn:adsk.eagle:library:348" deviceset="R-EU_" device="0207/7" package3d_urn="urn:adsk.eagle:package:23493/2" value="47">
-<attribute name="MF" value=""/>
-<attribute name="MPN" value=""/>
-<attribute name="OC_NEWARK" value="unknown"/>
-</part>
-<part name="P+3" library="supply1" library_urn="urn:adsk.eagle:library:371" deviceset="+15V" device=""/>
 <part name="D5" library="SparkFun-Connectors" library_urn="urn:adsk.eagle:library:513" deviceset="CONN_01" device="" package3d_urn="urn:adsk.eagle:package:38028/1" value="CONNECTOR 1x1 PIN">
 <attribute name="MF" value=""/>
@@
 <attribute name="MPN" x="35.56" y="119.38" size="1.778" layer="96" display="off"/>
 </instance>
-<instance part="R15" gate="G$1" x="187.96" y="190.5" smashed="yes">
-<attribute name="NAME" x="187.96" y="191.9986" size="1.778" layer="95" rot="R180" align="top-center"/>
-<attribute name="VALUE" x="187.96" y="189.23" size="1.778" layer="95" rot="R180" align="bottom-center"/>
-<attribute name="OC_NEWARK" x="187.96" y="190.5" size="1.778" layer="96" display="off"/>
-<attribute name="MF" x="187.96" y="190.5" size="1.778" layer="96" display="off"/>
-<attribute name="MPN" x="187.96" y="190.5" size="1.778" layer="96" display="off"/>
-</instance>
-<instance part="P+3" gate="1" x="198.12" y="187.96" smashed="yes" rot="R180">
-<attribute name="VALUE" x="200.66" y="190.5" size="1.778" layer="96" rot="R270"/>
-</instance>
 <instance part="D5" gate="G$1" x="10.16" y="81.28" smashed="yes">
 <attribute name="VALUE" x="7.62" y="76.454" size="1.778" layer="96" font="vector"/>
@@
 <wire x1="160.02" y1="177.8" x2="157.48" y2="177.8" width="0.1524" layer="91"/>
 <pinref part="P+10" gate="1" pin="+15V"/>
+<pinref part="STEER-SWITCH" gate="J$1" pin="3"/>
+<wire x1="152.4" y1="172.72" x2="157.48" y2="172.72" width="0.1524" layer="91"/>
+<wire x1="157.48" y1="177.8" x2="157.48" y2="172.72" width="0.1524" layer="91"/>
+<junction x="157.48" y="177.8"/>
 </segment>
 <segment>
@@
 <wire x1="160.02" y1="132.08" x2="157.48" y2="132.08" width="0.1524" layer="91"/>
 <pinref part="P+2" gate="1" pin="+15V"/>
+<pinref part="AUTO-SWITCH" gate="J$1" pin="3"/>
+<wire x1="157.48" y1="127" x2="152.4" y2="127" width="0.1524" layer="91"/>
+<wire x1="157.48" y1="132.08" x2="157.48" y2="127" width="0.1524" layer="91"/>
+<junction x="157.48" y="132.08"/>
 </segment>
 <segment>
@@
 <pinref part="P+7" gate="1" pin="+15V"/>
 <wire x1="157.48" y1="154.94" x2="160.02" y2="154.94" width="0.1524" layer="91"/>
-</segment>
-<segment>
-<pinref part="R15" gate="G$1" pin="2"/>
-<wire x1="193.04" y1="190.5" x2="198.12" y2="190.5" width="0.1524" layer="91"/>
-<pinref part="P+3" gate="1" pin="+15V"/>
+<pinref part="IMP-SWITCH" gate="J$1" pin="3"/>
+<wire x1="157.48" y1="149.86" x2="152.4" y2="149.86" width="0.1524" layer="91"/>
+<wire x1="157.48" y1="154.94" x2="157.48" y2="149.86" width="0.1524" layer="91"/>
+<junction x="157.48" y="154.94"/>
 </segment>
 </net>
@@
 </segment>
 </net>
-<net name="PO" class="0">
-<segment>
-<pinref part="R15" gate="G$1" pin="1"/>
-<wire x1="182.88" y1="190.5" x2="177.8" y2="190.5" width="0.1524" layer="91"/>
-<label x="177.8" y="190.5" size="1.778" layer="95"/>
-</segment>
-<segment>
-<pinref part="STEER-SWITCH" gate="J$1" pin="3"/>
-<wire x1="152.4" y1="172.72" x2="157.48" y2="172.72" width="0.1524" layer="91"/>
-<label x="152.4" y="172.72" size="1.778" layer="95"/>
-</segment>
-<segment>
-<pinref part="IMP-SWITCH" gate="J$1" pin="3"/>
-<wire x1="157.48" y1="149.86" x2="152.4" y2="149.86" width="0.1524" layer="91"/>
-<label x="152.4" y="149.86" size="1.778" layer="95"/>
-</segment>
-<segment>
-<pinref part="AUTO-SWITCH" gate="J$1" pin="3"/>
-<wire x1="157.48" y1="127" x2="152.4" y2="127" width="0.1524" layer="91"/>
-<label x="152.4" y="127" size="1.778" layer="95"/>
-</segment>
-</net>

Commit message: Add files via upload
Added pin A0 A1 A2 A3
Parts:
- added 1: CONNECTOR 1x2 PINS, SparkFun-Connectors:CONN_02
Connections:
- new net A0: 1.2, PCB1.A0
- new net A3: 0.1, PCB1.A3
- net A1: now also 1.1; no longer 0.2
- net A2: now also 0.2; no longer 0.1
Changed lines of the file:
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@@
 <part name="P+5" library="supply1" library_urn="urn:adsk.eagle:library:371" deviceset="+5V" device=""/>
 <part name="FRAME1" library="frames" library_urn="urn:adsk.eagle:library:229" deviceset="DOCFIELD" device=""/>
+<part name="1" library="SparkFun-Connectors" library_urn="urn:adsk.eagle:library:513" deviceset="CONN_02" device="" package3d_urn="urn:adsk.eagle:package:38039/1" value="CONNECTOR 1x2 PINS">
+<attribute name="MF" value=""/>
+<attribute name="MPN" value=""/>
+<attribute name="OC_NEWARK" value="unknown"/>
+</part>
 </parts>
 <sheets>
 <sheet>
 <plain>
-<wire x1="147.32" y1="274.32" x2="147.32" y2="259.08" width="0.1524" layer="97"/>
-<wire x1="198.12" y1="274.32" x2="198.12" y2="259.08" width="0.1524" layer="97"/>
-<wire x1="198.12" y1="274.32" x2="147.32" y2="274.32" width="0.1524" layer="97"/>
+<wire x1="147.32" y1="284.48" x2="147.32" y2="259.08" width="0.1524" layer="97"/>
+<wire x1="198.12" y1="284.48" x2="198.12" y2="259.08" width="0.1524" layer="97"/>
+<wire x1="198.12" y1="284.48" x2="147.32" y2="284.48" width="0.1524" layer="97"/>
 <wire x1="198.12" y1="259.08" x2="147.32" y2="259.08" width="0.1524" layer="97"/>
 <wire x1="205.74" y1="114.3" x2="132.08" y2="114.3" width="0.1524" layer="97"/>
@@
 <attribute name="DRAWING_NAME" x="127" y="82.55" size="2.54" layer="94"/>
 </instance>
+<instance part="1" gate="G$1" x="170.18" y="276.86" smashed="yes">
+<attribute name="NAME" x="167.64" y="282.448" size="1.778" layer="95" font="vector"/>
+<attribute name="OC_NEWARK" x="170.18" y="276.86" size="1.778" layer="96" display="off"/>
+<attribute name="MF" x="170.18" y="276.86" size="1.778" layer="96" display="off"/>
+<attribute name="MPN" x="170.18" y="276.86" size="1.778" layer="96" display="off"/>
+</instance>
 </instances>
 <busses>
@@
 <net name="A1" class="0">
 <segment>
+<pinref part="PCB1" gate="G$1" pin="A1"/>
+<wire x1="190.5" y1="213.36" x2="195.58" y2="213.36" width="0.1524" layer="91"/>
+<label x="193.04" y="213.36" size="1.778" layer="95"/>
+</segment>
+<segment>
+<pinref part="1" gate="G$1" pin="1"/>
+<wire x1="177.8" y1="276.86" x2="180.34" y2="276.86" width="0.1524" layer="91"/>
+<label x="177.8" y="276.86" size="1.778" layer="95"/>
+</segment>
+</net>
+<net name="A2" class="0">
+<segment>
+<pinref part="PCB1" gate="G$1" pin="A2"/>
+<wire x1="190.5" y1="215.9" x2="195.58" y2="215.9" width="0.1524" layer="91"/>
+<label x="193.04" y="215.9" size="1.778" layer="95"/>
+</segment>
+<segment>
 <pinref part="0" gate="G$1" pin="2"/>
 <wire x1="177.8" y1="266.7" x2="180.34" y2="266.7" width="0.1524" layer="91"/>
 <label x="177.8" y="266.7" size="1.778" layer="95"/>
 </segment>
-<segment>
-<pinref part="PCB1" gate="G$1" pin="A1"/>
-<wire x1="190.5" y1="213.36" x2="195.58" y2="213.36" width="0.1524" layer="91"/>
-<label x="193.04" y="213.36" size="1.778" layer="95"/>
-</segment>
-</net>
-<net name="A2" class="0">
+</net>
+<net name="A0" class="0">
+<segment>
+<pinref part="1" gate="G$1" pin="2"/>
+<wire x1="177.8" y1="279.4" x2="180.34" y2="279.4" width="0.1524" layer="91"/>
+<label x="177.8" y="279.4" size="1.778" layer="95"/>
+</segment>
+<segment>
+<pinref part="PCB1" gate="G$1" pin="A0"/>
+<wire x1="190.5" y1="210.82" x2="195.58" y2="210.82" width="0.1524" layer="91"/>
+<label x="193.04" y="210.82" size="1.778" layer="95"/>
+</segment>
+</net>
+<net name="A3" class="0">
 <segment>
 <pinref part="0" gate="G$1" pin="1"/>
@@
 </segment>
 <segment>
-<pinref part="PCB1" gate="G$1" pin="A2"/>
-<wire x1="190.5" y1="215.9" x2="195.58" y2="215.9" width="0.1524" layer="91"/>
-<label x="193.04" y="215.9" size="1.778" layer="95"/>
-</segment>
-</net>
+<pinref part="PCB1" gate="G$1" pin="A3"/>
+<wire x1="190.5" y1="218.44" x2="195.58" y2="218.44" width="0.1524" layer="91"/>
+<label x="193.04" y="218.44" size="1.778" layer="95"/>
+</segment>
+</net>

Commit message: Add files via upload
Parts:
- removed IC2: MMA8452Q, MMA8452Q:MMA8452Q
- added R15: 1k, resistor:R-EU_0207/7
- added U$13: MMA8542Q, #MMA8542Q:MMA8542Q
- 0, 1: device SparkFun-Connectors:CONN_02 -> SparkFun-Connectors:CONN_03
- D5: device SparkFun-Connectors:CONN_01 -> SparkFun-Connectors:CONN_02
Connections:
- new net D5.: D5.1, R15.1
- net +3V3: now also U$13.3.3V; no longer IC2.3.3V
- net A0: now also 1.3; no longer 1.2
- net A1: now also 1.2; no longer 1.1
- net D5: now also R15.2; no longer D5.1
- net GND: now also 0.3, 1.1, D5.2, U$13.GND; no longer IC2.GND
- net N$1: now also U$13.SDA; no longer IC2.SDA
- net N$9: now also U$13.SCL; no longer IC2.SCL
Other:
- moved on the sheet: INT

Commit message: Add files via upload
Adding jumper SAO
Parts:
- added SAO: CONNECTOR 1x2 PINS, SparkFun-Connectors:CONN_02
Connections:
- new net N$23: MMA8542.SAO, SAO.2
- net GND: now also SAO.1
Other:
- moved on the sheet: C6, C9

Commit message: Add files via upload
Small edit - silkscreen
Parts:
- removed SAO: CONNECTOR 1x2 PINS, SparkFun-Connectors:CONN_02
Connections:
- removed net N$23: MMA8542.SAO, SAO.2
- new net SAO: MMA8542.SAO
- net GND: no longer SAO.1
Changed lines of the file:
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@@
-<attribute name="OC_NEWARK" value="unknown"/>
-</part>
-<part name="SAO" library="SparkFun-Connectors" library_urn="urn:adsk.eagle:library:513" deviceset="CONN_02" device="" package3d_urn="urn:adsk.eagle:package:38039/1" value="CONNECTOR 1x2 PINS">
-<attribute name="MF" value=""/>
-<attribute name="MPN" value=""/>
 <attribute name="OC_NEWARK" value="unknown"/>
 </part>
@@
 <attribute name="MPN" x="27.94" y="81.28" size="1.778" layer="96" display="off"/>
 </instance>
-<instance part="SAO" gate="G$1" x="10.16" y="127" smashed="yes">
-<attribute name="NAME" x="10.16" y="133.858" size="1.778" layer="95" font="vector" align="center"/>
-<attribute name="OC_NEWARK" x="10.16" y="127" size="1.778" layer="96" display="off"/>
-<attribute name="MF" x="10.16" y="127" size="1.778" layer="96" display="off"/>
-<attribute name="MPN" x="10.16" y="127" size="1.778" layer="96" display="off"/>
-</instance>
 </instances>
 <busses>
@@
 <wire x1="160.02" y1="274.32" x2="162.56" y2="274.32" width="0.1524" layer="91"/>
 <label x="160.02" y="274.32" size="1.778" layer="95"/>
-</segment>
-<segment>
-<pinref part="SAO" gate="G$1" pin="1"/>
-<wire x1="17.78" y1="127" x2="17.78" y2="119.38" width="0.1524" layer="91"/>
-<wire x1="17.78" y1="119.38" x2="7.62" y2="119.38" width="0.1524" layer="91"/>
-<label x="7.62" y="119.38" size="1.778" layer="95"/>
 </segment>
 </net>
@@
 </segment>
 </net>
-<net name="N$23" class="0">
+<net name="SAO" class="0">
 <segment>
 <pinref part="MMA8542" gate="G$1" pin="SAO"/>
-<pinref part="SAO" gate="G$1" pin="2"/>
 <wire x1="17.78" y1="129.54" x2="22.86" y2="129.54" width="0.1524" layer="91"/>
 </segment>
