File: AutoSteerAiO (BNO-MMA connector)/AutoSteerAiO (BNO-MMA connector).sch (EAGLE design)
At the start: 85 parts, among them K4 CB1A-P-12V, T1 BC547, U1 VX7805-1000

Commit message: Add files via upload
Parts:
- ENCODER: device SparkFun-Connectors:CONN_04 -> SparkFun-Connectors:CONN_03
Connections:
- removed net N$31: ENCODER.3, OK4.C
- removed net N$32: D5.C, ENCODER.4
- new net N$19: D5.C, ENCODER.3
- new net N$20: ENCODER.2, OK4.C
- net +15V: no longer ENCODER.1
- net GND: now also ENCODER.1; no longer ENCODER.2
Changed lines of the file:
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@@
 <attribute name="OC_NEWARK" value="unknown"/>
 </part>
-<part name="ENCODER" library="SparkFun-Connectors" library_urn="urn:adsk.eagle:library:513" deviceset="CONN_04" device="" package3d_urn="urn:adsk.eagle:package:38085/1" value="CONNECTOR 1x3 PINS">
+<part name="ENCODER" library="SparkFun-Connectors" library_urn="urn:adsk.eagle:library:513" deviceset="CONN_03" device="" package3d_urn="urn:adsk.eagle:package:38063/1" value="CONNECTOR 1x3 PINS">
 <attribute name="MF" value=""/>
 <attribute name="MPN" value=""/>
@@
 <attribute name="MPN" x="195.58" y="170.18" size="1.778" layer="96" display="off"/>
 </instance>
-<instance part="ENCODER" gate="G$1" x="147.32" y="177.8" smashed="yes">
-<attribute name="NAME" x="147.32" y="187.198" size="1.778" layer="95" font="vector" align="center"/>
-<attribute name="OC_NEWARK" x="147.32" y="177.8" size="1.778" layer="96" display="off"/>
-<attribute name="MF" x="147.32" y="177.8" size="1.778" layer="96" display="off"/>
-<attribute name="MPN" x="147.32" y="177.8" size="1.778" layer="96" display="off"/>
+<instance part="ENCODER" gate="J$1" x="144.78" y="180.34" smashed="yes">
+<attribute name="NAME" x="144.78" y="189.738" size="1.778" layer="95" font="vector" align="center"/>
+<attribute name="OC_NEWARK" x="144.78" y="180.34" size="1.778" layer="96" display="off"/>
+<attribute name="MF" x="144.78" y="180.34" size="1.778" layer="96" display="off"/>
+<attribute name="MPN" x="144.78" y="180.34" size="1.778" layer="96" display="off"/>
 </instance>
 <instance part="R22" gate="G$1" x="195.58" y="185.42" smashed="yes">
@@
 </segment>
 <segment>
-<pinref part="ENCODER" gate="G$1" pin="2"/>
-<wire x1="152.4" y1="177.8" x2="165.1" y2="177.8" width="0.1524" layer="91"/>
-<pinref part="GND22" gate="1" pin="GND"/>
-</segment>
-<segment>
 <pinref part="GND25" gate="1" pin="GND"/>
 <pinref part="5V" gate="G$1" pin="1"/>
@@
 <wire x1="45.72" y1="83.82" x2="38.1" y2="83.82" width="0.1524" layer="91"/>
 <label x="38.1" y="83.82" size="1.778" layer="95"/>
+</segment>
+<segment>
+<pinref part="GND22" gate="1" pin="GND"/>
+<pinref part="ENCODER" gate="J$1" pin="1"/>
+<wire x1="165.1" y1="177.8" x2="152.4" y2="177.8" width="0.1524" layer="91"/>
 </segment>
 </net>
@@
 <wire x1="157.48" y1="165.1" x2="157.48" y2="160.02" width="0.1524" layer="91"/>
 <junction x="157.48" y="165.1"/>
-<pinref part="ENCODER" gate="G$1" pin="1"/>
-<wire x1="152.4" y1="160.02" x2="152.4" y2="175.26" width="0.1524" layer="91"/>
-<junction x="152.4" y="160.02"/>
 </segment>
 <segment>
@@
 </segment>
 </net>
-<net name="N$31" class="0">
-<segment>
-<pinref part="OK4" gate="A" pin="C"/>
-<pinref part="ENCODER" gate="G$1" pin="3"/>
-<wire x1="170.18" y1="180.34" x2="152.4" y2="180.34" width="0.1524" layer="91"/>
-</segment>
-</net>
-<net name="N$32" class="0">
-<segment>
-<pinref part="ENCODER" gate="G$1" pin="4"/>
-<wire x1="154.94" y1="182.88" x2="152.4" y2="182.88" width="0.1524" layer="91"/>
-<pinref part="D5" gate="1" pin="C"/>
-</segment>
-</net>
 <net name="PWM2" class="0">
 <segment>
@@
 </segment>
 </net>
+<net name="N$19" class="0">
+<segment>
+<pinref part="D5" gate="1" pin="C"/>
+<pinref part="ENCODER" gate="J$1" pin="3"/>
+<wire x1="154.94" y1="182.88" x2="152.4" y2="182.88" width="0.1524" layer="91"/>
+</segment>
+</net>
+<net name="N$20" class="0">
+<segment>
+<pinref part="ENCODER" gate="J$1" pin="2"/>
+<pinref part="OK4" gate="A" pin="C"/>
+<wire x1="152.4" y1="180.34" x2="170.18" y2="180.34" width="0.1524" layer="91"/>
+</segment>
+</net>

Commit message: Add files via upload
Parts:
- K4: device relay:CB1A-P-12V -> #relay:CB1A-P-12V; OC_NEWARK unknown -> (none)
Changed lines of the file:
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@@
 <part name="P+11" library="supply1" library_urn="urn:adsk.eagle:library:371" deviceset="+5V" device=""/>
 <part name="OK1" library="#optocoupler" deviceset="4N33" device="" package3d_urn="urn:adsk.eagle:package:21942/1"/>
-<part name="K4" library="relay" library_urn="urn:adsk.eagle:library:339" deviceset="CB*" device="" package3d_urn="urn:adsk.eagle:package:24437/1" technology="1A-P-12V">
-<attribute name="MF" value=""/>
-<attribute name="MPN" value=""/>
-<attribute name="OC_NEWARK" value="unknown"/>
-</part>
+<part name="K4" library="#relay" deviceset="CB*" device="" technology="1A-P-12V"/>
 <part name="OK2" library="#optocoupler" deviceset="4N33" device="" package3d_urn="urn:adsk.eagle:package:21942/1"/>
 <part name="OK3" library="#optocoupler" deviceset="4N33" device="" package3d_urn="urn:adsk.eagle:package:21942/1"/>
