File: AutoSteerAiO (BNO-MMA connector)/AutoSteerAiO (BNO-MMA connector).sch (EAGLE design)
At the start: 85 parts, among them K4 CB1A-P-12V, T1 BC547, U1 VX7805-1000

Commit message: Add files via upload
Parts:
- IBT2: device SparkFun-Connectors:CONN_04X2 -> pinhead:PINHD-2X4
Changed lines of the file:
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@@
 <?xml version="1.0" encoding="utf-8"?>
 <!DOCTYPE eagle SYSTEM "eagle.dtd">
-<eagle version="9.3.2">
+<eagle version="9.4.0">
 <drawing>
 <settings>
@@
 <attribute name="OC_NEWARK" value="unknown"/>
 </part>
-<part name="IBT2" library="SparkFun-Connectors" library_urn="urn:adsk.eagle:library:513" deviceset="CONN_04X2" device="" package3d_urn="urn:adsk.eagle:package:38103/1">
+<part name="IBT2" library="pinhead" library_urn="urn:adsk.eagle:library:325" deviceset="PINHD-2X4" device="" package3d_urn="urn:adsk.eagle:package:22461/2">
 <attribute name="MF" value=""/>
 <attribute name="MPN" value=""/>
@@
 <attribute name="MPN" x="73.66" y="270.51" size="1.778" layer="96" display="off"/>
 </instance>
-<instance part="IBT2" gate="G$1" x="53.34" y="99.06" smashed="yes">
+<instance part="IBT2" gate="A" x="53.34" y="99.06" smashed="yes">
 <attribute name="VALUE" x="49.53" y="91.694" size="1.778" layer="96" font="vector"/>
 <attribute name="NAME" x="49.276" y="107.188" size="1.778" layer="95" font="vector"/>
@@
 </segment>
 <segment>
-<pinref part="IBT2" gate="G$1" pin="7"/>
-<wire x1="45.72" y1="96.52" x2="40.64" y2="96.52" width="0.1524" layer="91"/>
+<pinref part="IBT2" gate="A" pin="7"/>
+<wire x1="50.8" y1="96.52" x2="40.64" y2="96.52" width="0.1524" layer="91"/>
 <label x="40.64" y="96.52" size="1.778" layer="95"/>
 </segment>
@@
 </segment>
 <segment>
-<pinref part="IBT2" gate="G$1" pin="8"/>
-<wire x1="60.96" y1="96.52" x2="66.04" y2="96.52" width="0.1524" layer="91"/>
+<pinref part="IBT2" gate="A" pin="8"/>
+<wire x1="58.42" y1="96.52" x2="66.04" y2="96.52" width="0.1524" layer="91"/>
 <label x="60.96" y="96.52" size="1.778" layer="95"/>
 </segment>
@@
 </segment>
 <segment>
-<pinref part="IBT2" gate="G$1" pin="3"/>
-<wire x1="45.72" y1="101.6" x2="43.18" y2="101.6" width="0.1524" layer="91"/>
+<pinref part="IBT2" gate="A" pin="3"/>
+<wire x1="50.8" y1="101.6" x2="43.18" y2="101.6" width="0.1524" layer="91"/>
 <label x="43.18" y="101.6" size="1.778" layer="95"/>
 </segment>
 <segment>
-<pinref part="IBT2" gate="G$1" pin="4"/>
-<wire x1="60.96" y1="101.6" x2="63.5" y2="101.6" width="0.1524" layer="91"/>
+<pinref part="IBT2" gate="A" pin="4"/>
+<wire x1="58.42" y1="101.6" x2="63.5" y2="101.6" width="0.1524" layer="91"/>
 <label x="60.96" y="101.6" size="1.778" layer="95"/>
 </segment>
@@
 <net name="PWM1" class="0">
 <segment>
-<pinref part="IBT2" gate="G$1" pin="2"/>
-<wire x1="60.96" y1="104.14" x2="68.58" y2="104.14" width="0.1524" layer="91"/>
+<pinref part="IBT2" gate="A" pin="2"/>
+<wire x1="58.42" y1="104.14" x2="68.58" y2="104.14" width="0.1524" layer="91"/>
 <label x="60.96" y="104.14" size="1.778" layer="95"/>
 </segment>
@@
 <net name="PWM2" class="0">
 <segment>
-<pinref part="IBT2" gate="G$1" pin="1"/>
-<wire x1="45.72" y1="104.14" x2="38.1" y2="104.14" width="0.1524" layer="91"/>
+<pinref part="IBT2" gate="A" pin="1"/>
+<wire x1="50.8" y1="104.14" x2="38.1" y2="104.14" width="0.1524" layer="91"/>
 <label x="38.1" y="104.14" size="1.778" layer="95"/>
 </segment>
