File: AutoSteerAiO/AutoSteerAIO.brd (EAGLE design)
At the start: 114.3 x 108 mm, 91 parts, among them K4 CB1A-P-12V, U1 VX7805-1000

Commit message: Add files via upload
Parts:
- added RST: CONNECTOR 1x2 PINS, SparkFun-Connectors:1X02
- moved C5 2.84 mm to (16.5, 94.0)
- moved C10 2.84 mm to (7.44, 72.4)
- moved C15 2.84 mm to (10.2, 94.0)
- moved C3 2.84 mm to (7.43, 88.9)
- moved C6 2.84 mm to (19.1, 88.3)
- moved C7 2.84 mm to (19.1, 73.0)
- moved U1 2.84 mm to (7.62, 80.6)
- moved 7805 2.84 mm to (19.1, 80.6)
- moved 0 1.27 mm to (41.3, 5.08)
- moved 1 1.27 mm to (48.9, 5.08)
- moved 5V3 1.27 mm to (38.7, 5.08)
- moved J1 1.27 mm to (56.5, 5.08)
Connections:
- new net RST: PCB1.RST., RST.2
- net GND: now also RST.1
Routing:
- net RST: track 0.00 -> 8.07 mm
- net GND: track 490.0 -> 498.0 mm
- net A+5V: track 111.4 -> 109.6 mm
- net N$26: track 54.1 -> 55.4 mm
- net +5V: track 350.3 -> 351.0 mm
- net A6: track 42.1 -> 41.6 mm
- net A3: track 35.2 -> 34.6 mm
- net A2: track 34.1 -> 33.5 mm
- net A1: track 32.9 -> 32.4 mm
- net A0: track 31.8 -> 31.3 mm
