File: AutoSteerAiO/AutoSteerAIO.brd (EAGLE design)
At the start: 114.3 x 108 mm, 92 parts, among them K4 CB1A-P-12V, U1 VX7805-1000

Commit message: Add files via upload
Parts:
- moved D3 17.3 mm to (42.5, 81.9)
- moved D2 17.3 mm to (48.9, 79.4)
- moved R16 2.54 mm to (55.9, 68.6)
- moved 15V1 1.27 mm to (78.7, 55.9)
- moved 15V2 1.27 mm to (87.6, 55.9)
- moved LED1 1.27 mm to (48.3, 66.0)
- moved LED2 1.27 mm to (63.5, 66.0)
Routing:
- net +15V: track 252.3 -> 277.3 mm
- net GND: track 498.0 -> 484.1 mm, vias 101 -> 93
- net N$26: track 55.4 -> 59.0 mm
- net A+5V: track 109.6 -> 107.3 mm
- net N$13: track 6.66 -> 5.39 mm
- net N$14: track 4.34 -> 3.81 mm
Other:
- board text added: "Power out"
- board text removed: "Power"
- board text removed: "Set the Diode and Capacitor to the bottom if you want to put the module without headres directly on the PCB But make sure there is no contact on the top layer with Ethernet module!"
